File: PCB/V101/Index.kicad_sch (KiCad schematic)
At the start: 0 parts

Commit message: Updated Layout
Other:
- note added: "Mechanical Parts"
Changed lines of the file:
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@@
 		)
 	)
-	(text "Debug"
+	(text "Mechanical Parts"
 		(exclude_from_sim no)
-		(at 52.578 147.066 0)
+		(at 73.152 146.304 0)
 		(effects
 			(font
