File: PCB/V101/Interface-CANFD.kicad_sch (KiCad schematic)
At the start: 0 parts

Commit message: Updated Layout
Parts:
- added C901: 4700pF, Capacitor_SMD:C_0603_1608Metric_Pad1.08x0.95mm_HandSolder, symbol Device:C
- added C902: 0.1uF, Capacitor_SMD:C_0603_1608Metric_Pad1.08x0.95mm_HandSolder, symbol Device:C
- added D901, D902: SMAJ7.0CA, Diode_SMD:D_SMA, symbol Diode:SMAJ7.0CA
- added J901: Conn_01x04, Connector_JST:JST_PH_S4B-PH-K_1x04_P2.00mm_Horizontal, symbol Connector_Generic:Conn_01x04
- added R901, R902: 60R, Resistor_SMD:R_0603_1608Metric_Pad0.98x0.95mm_HandSolder, symbol Device:R
- added U901: MCP2557FD-xMF, Package_DFN_QFN:DFN-8-1EP_3x3mm_P0.65mm_EP1.55x2.4mm, symbol Interface_CAN_LIN:MCP2557FD-xMF
Connections:
- new net: D902.2 (A2), J901.2 (Pin_2), R902.2, U901.6 (CANL)
- new net: D901.2 (A2), J901.3 (Pin_3), R901.1, U901.7 (CANH)
- new net: C901.1, R901.2, R902.1
- new net +5V: C902.1, U901.3 (VDD)
- new net CAN1_RXD: U901.4 (RXD)
- new net CAN1_TXD: U901.1 (TXD)
- new net CAN_TRX_S: U901.8 (S)
- new net GND: C901.2, C902.2, D901.1 (A1), D902.1 (A1), J901.4 (Pin_4), U901.2 (VSS), U901.9 (VSS)
- new net VDD: J901.1 (Pin_1)
