File: PCB/V101/Power.kicad_sch (KiCad schematic)
At the start: 13 parts, among them U601 TPS54302

Commit message: Updated Layout
Parts:
- C601: renamed from C604; footprint (none) -> Capacitor_SMD:C_0603_1608Metric_Pad1.08x0.95mm_HandSolder
- C602: renamed from C605; footprint (none) -> Capacitor_SMD:C_0603_1608Metric_Pad1.08x0.95mm_HandSolder
- C603: renamed from C601; footprint (none) -> Capacitor_SMD:C_0603_1608Metric_Pad1.08x0.95mm_HandSolder
- C604: renamed from C602; footprint (none) -> Capacitor_SMD:C_0603_1608Metric_Pad1.08x0.95mm_HandSolder
- C605: renamed from C606; footprint (none) -> Capacitor_SMD:C_0603_1608Metric_Pad1.08x0.95mm_HandSolder
- C606: renamed from C607; footprint (none) -> Capacitor_SMD:C_0603_1608Metric_Pad1.08x0.95mm_HandSolder
- L601: footprint (none) -> Inductor_SMD:L_APV_ANR5045
- R601: renamed from R603; footprint (none) -> Resistor_SMD:R_0603_1608Metric_Pad0.98x0.95mm_HandSolder
- R602: renamed from R604; footprint (none) -> Resistor_SMD:R_0603_1608Metric_Pad0.98x0.95mm_HandSolder
- R603: renamed from R601; footprint (none) -> Resistor_SMD:R_0603_1608Metric_Pad0.98x0.95mm_HandSolder
- R604: renamed from R605; footprint (none) -> Resistor_SMD:R_0603_1608Metric_Pad0.98x0.95mm_HandSolder
- R605: renamed from R602; footprint (none) -> Resistor_SMD:R_0603_1608Metric_Pad0.98x0.95mm_HandSolder
Changed lines of the file:
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@@
 		(dnp no)
 		(fields_autoplaced yes)
-		(property "Reference" "C601"
+		(property "Reference" "C603"
 			(at 152.4 29.21 90)
 			(effects
@@
 			)
 		)
-		(property "Footprint" ""
+		(property "Footprint" "Capacitor_SMD:C_0603_1608Metric_Pad1.08x0.95mm_HandSolder"
 			(at 156.21 35.8648 0)
 			(effects
@@
 			(project ""
 				(path "/2bb6e42f-287e-4818-b6e1-26da2df0523c/c8e95473-f617-4ba5-be50-45b0179e07ec"
-					(reference "C601")
+					(reference "C603")
 					(unit 1)
 				)
@@
 		(dnp no)
 		(fields_autoplaced yes)
-		(property "Reference" "C605"
+		(property "Reference" "C602"
 			(at 95.25 50.7999 0)
 			(effects
@@
 			)
 		)
-		(property "Footprint" ""
+		(property "Footprint" "Capacitor_SMD:C_0603_1608Metric_Pad1.08x0.95mm_HandSolder"
 			(at 92.4052 55.88 0)
 			(effects
@@
 			(project "V101"
 				(path "/2bb6e42f-287e-4818-b6e1-26da2df0523c/c8e95473-f617-4ba5-be50-45b0179e07ec"
-					(reference "C605")
+					(reference "C602")
 					(unit 1)
 				)
@@
 		(dnp no)
 		(fields_autoplaced yes)
-		(property "Reference" "#PWR0608"
+		(property "Reference" "#PWR0606"
 			(at 191.77 73.66 0)
 			(effects
@@
 			(project "V101"
 				(path "/2bb6e42f-287e-4818-b6e1-26da2df0523c/c8e95473-f617-4ba5-be50-45b0179e07ec"
-					(reference "#PWR0608")
+					(reference "#PWR0606")
 					(unit 1)
 				)
@@
 		(dnp no)
 		(fields_autoplaced yes)
-		(property "Reference" "C602"
+		(property "Reference" "C604"
 			(at 182.88 53.3399 0)
 			(effects
@@
 			)
 		)
-		(property "Footprint" ""
+		(property "Footprint" "Capacitor_SMD:C_0603_1608Metric_Pad1.08x0.95mm_HandSolder"
 			(at 180.0352 58.42 0)
 			(effects
@@
 			(project ""
 				(path "/2bb6e42f-287e-4818-b6e1-26da2df0523c/c8e95473-f617-4ba5-be50-45b0179e07ec"
-					(reference "C602")
+					(reference "C604")
 					(unit 1)
 				)
@@
 		(dnp no)
 		(fields_autoplaced yes)
-		(property "Reference" "#PWR0605"
+		(property "Reference" "#PWR0602"
 			(at 91.44 69.85 0)
 			(effects
@@
 			(project "V101"
 				(path "/2bb6e42f-287e-4818-b6e1-26da2df0523c/c8e95473-f617-4ba5-be50-45b0179e07ec"
-					(reference "#PWR0605")
+					(reference "#PWR0602")
 					(unit 1)
 				)
@@
 		(dnp no)
 		(fields_autoplaced yes)
-		(property "Reference" "R601"
+		(property "Reference" "R603"
 			(at 224.79 53.3399 0)
 			(effects
@@
 			)
 		)
-		(property "Footprint" ""
+		(property "Footprint" "Resistor_SMD:R_0603_1608Metric_Pad0.98x0.95mm_HandSolder"
 			(at 220.472 54.61 90)
 			(effects
@@
 			(project ""
 				(path "/2bb6e42f-287e-4818-b6e1-26da2df0523c/c8e95473-f617-4ba5-be50-45b0179e07ec"
-					(reference "R601")
+					(reference "R603")
 					(unit 1)
 				)
@@
 		(dnp no)
 		(fields_autoplaced yes)
-		(property "Reference" "C607"
+		(property "Reference" "C606"
 			(at 214.63 67.3099 0)
 			(effects
@@
 			)
 		)
-		(property "Footprint" ""
+		(property "Footprint" "Capacitor_SMD:C_0603_1608Metric_Pad1.08x0.95mm_HandSolder"
 			(at 211.7852 72.39 0)
 			(effects
@@
 			(project "V101"
 				(path "/2bb6e42f-287e-4818-b6e1-26da2df0523c/c8e95473-f617-4ba5-be50-45b0179e07ec"
-					(reference "C607")
+					(reference "C606")
 					(unit 1)
 				)
@@
 		(dnp no)
 		(fields_autoplaced yes)
-		(property "Reference" "R603"
+		(property "Reference" "R601"
 			(at 106.68 50.7999 0)
 			(effects
@@
 			)
 		)
-		(property "Footprint" ""
+		(property "Footprint" "Resistor_SMD:R_0603_1608Metric_Pad0.98x0.95mm_HandSolder"
 			(at 102.362 52.07 90)
 			(effects
@@
 			(project "V101"
 				(path "/2bb6e42f-287e-4818-b6e1-26da2df0523c/c8e95473-f617-4ba5-be50-45b0179e07ec"
-					(reference "R603")
+					(reference "R601")
 					(unit 1)
 				)
@@
 		(dnp no)
 		(fields_autoplaced yes)
-		(property "Reference" "#PWR0601"
+		(property "Reference" "#PWR0604"
 			(at 132.08 68.58 0)
 			(effects
@@
 			(project ""
 				(path "/2bb6e42f-287e-4818-b6e1-26da2df0523c/c8e95473-f617-4ba5-be50-45b0179e07ec"
-					(reference "#PWR0601")
+					(reference "#PWR0604")
 					(unit 1)
 				)
@@
 		(dnp no)
 		(fields_autoplaced yes)
-		(property "Reference" "#PWR0607"
+		(property "Reference" "#PWR0605"
 			(at 179.07 73.66 0)
 			(effects
@@
 			(project "V101"
 				(path "/2bb6e42f-287e-4818-b6e1-26da2df0523c/c8e95473-f617-4ba5-be50-45b0179e07ec"
-					(reference "#PWR0607")
+					(reference "#PWR0605")
 					(unit 1)
 				)
@@
 		(dnp no)
 		(fields_autoplaced yes)
-		(property "Reference" "#PWR0606"
+		(property "Reference" "#PWR0603"
 			(at 104.14 78.74 0)
 			(effects
@@
 			(project "V101"
 				(path "/2bb6e42f-287e-4818-b6e1-26da2df0523c/c8e95473-f617-4ba5-be50-45b0179e07ec"
-					(reference "#PWR0606")
+					(reference "#PWR0603")
 					(unit 1)
 				)
@@
 		(dnp no)
 		(fields_autoplaced yes)
-		(property "Reference" "R605"
+		(property "Reference" "R604"
 			(at 224.79 67.3099 0)
 			(effects
@@
 			)
 		)
-		(property "Footprint" ""
+		(property "Footprint" "Resistor_SMD:R_0603_1608Metric_Pad0.98x0.95mm_HandSolder"
 			(at 220.472 68.58 90)
 			(effects
@@
 			(project "V101"
 				(path "/2bb6e42f-287e-4818-b6e1-26da2df0523c/c8e95473-f617-4ba5-be50-45b0179e07ec"
-					(reference "R605")
+					(reference "R604")
 					(unit 1)
 				)
@@
 		(dnp no)
 		(fields_autoplaced yes)
-		(property "Reference" "R602"
+		(property "Reference" "R605"
 			(at 224.79 81.2799 0)
 			(effects
@@
 			)
 		)
-		(property "Footprint" ""
+		(property "Footprint" "Resistor_SMD:R_0603_1608Metric_Pad0.98x0.95mm_HandSolder"
 			(at 220.472 82.55 90)
 			(effects
@@
 			(project "V101"
 				(path "/2bb6e42f-287e-4818-b6e1-26da2df0523c/c8e95473-f617-4ba5-be50-45b0179e07ec"
-					(reference "R602")
+					(reference "R605")
 					(unit 1)
 				)
@@
 		(dnp no)
 		(fields_autoplaced yes)
-		(property "Reference" "C606"
+		(property "Reference" "C605"
 			(at 195.58 53.3399 0)
 			(effects
@@
 			)
 		)
-		(property "Footprint" ""
+		(property "Footprint" "Capacitor_SMD:C_0603_1608Metric_Pad1.08x0.95mm_HandSolder"
 			(at 192.7352 58.42 0)
 			(effects
@@
 			(project "V101"
 				(path "/2bb6e42f-287e-4818-b6e1-26da2df0523c/c8e95473-f617-4ba5-be50-45b0179e07ec"
-					(reference "C606")
+					(reference "C605")
 					(unit 1)
 				)
@@
 			)
 		)
-		(property "Footprint" ""
+		(property "Footprint" "Inductor_SMD:L_APV_ANR5045"
 			(at 166.37 36.83 0)
 			(effects
@@
 		(dnp no)
 		(fields_autoplaced yes)
-		(property "Reference" "R604"
+		(property "Reference" "R602"
 			(at 106.68 64.7699 0)
 			(effects
@@
 			)
 		)
-		(property "Footprint" ""
+		(property "Footprint" "Resistor_SMD:R_0603_1608Metric_Pad0.98x0.95mm_HandSolder"
 			(at 102.362 66.04 90)
 			(effects
@@
 			(project "V101"
 				(path "/2bb6e42f-287e-4818-b6e1-26da2df0523c/c8e95473-f617-4ba5-be50-45b0179e07ec"
-					(reference "R604")
+					(reference "R602")
 					(unit 1)
 				)
@@
 		(dnp no)
 		(fields_autoplaced yes)
-		(property "Reference" "#PWR0604"
+		(property "Reference" "#PWR0601"
 			(at 78.74 69.85 0)
 			(effects
@@
 			(project "V101"
 				(path "/2bb6e42f-287e-4818-b6e1-26da2df0523c/c8e95473-f617-4ba5-be50-45b0179e07ec"
-					(reference "#PWR0604")
+					(reference "#PWR0601")
 					(unit 1)
 				)
@@
 		(dnp no)
 		(fields_autoplaced yes)
-		(property "Reference" "#PWR0602"
+		(property "Reference" "#PWR0607"
 			(at 222.25 95.25 0)
 			(effects
@@
 			(project "V101"
 				(path "/2bb6e42f-287e-4818-b6e1-26da2df0523c/c8e95473-f617-4ba5-be50-45b0179e07ec"
-					(reference "#PWR0602")
+					(reference "#PWR0607")
 					(unit 1)
 				)
@@
 		(dnp no)
 		(fields_autoplaced yes)
-		(property "Reference" "C604"
+		(property "Reference" "C601"
 			(at 82.55 50.7999 0)
 			(effects
@@
 			)
 		)
-		(property "Footprint" ""
+		(property "Footprint" "Capacitor_SMD:C_0603_1608Metric_Pad1.08x0.95mm_HandSolder"
 			(at 79.7052 55.88 0)
 			(effects
@@
 			(project "V101"
 				(path "/2bb6e42f-287e-4818-b6e1-26da2df0523c/c8e95473-f617-4ba5-be50-45b0179e07ec"
-					(reference "C604")
-					(unit 1)
-				)
+					(reference "C601")
+					(unit 1)
+				)
