File: PCB/V101/Sensors.kicad_sch (KiCad schematic)
At the start: 10 parts, among them U701 BME280, U702 BME280

Commit message: Updated Layout
Parts:
- C701: renamed from C702; footprint (none) -> Capacitor_SMD:C_0603_1608Metric_Pad1.08x0.95mm_HandSolder
- C702: renamed from C703; footprint (none) -> Capacitor_SMD:C_0603_1608Metric_Pad1.08x0.95mm_HandSolder
- C703: renamed from C701; footprint (none) -> Capacitor_SMD:C_0603_1608Metric_Pad1.08x0.95mm_HandSolder
- C704: footprint (none) -> Capacitor_SMD:C_0603_1608Metric_Pad1.08x0.95mm_HandSolder
- R701, R704: footprint (none) -> Resistor_SMD:R_0603_1608Metric_Pad0.98x0.95mm_HandSolder
- R702: renamed from R703; footprint (none) -> Resistor_SMD:R_0603_1608Metric_Pad0.98x0.95mm_HandSolder
- R703: renamed from R702; footprint (none) -> Resistor_SMD:R_0603_1608Metric_Pad0.98x0.95mm_HandSolder
Changed lines of the file:
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@@
 		(dnp no)
 		(fields_autoplaced yes)
-		(property "Reference" "R703"
+		(property "Reference" "R702"
 			(at 180.34 120.6499 0)
 			(effects
@@
 			)
 		)
-		(property "Footprint" ""
+		(property "Footprint" "Resistor_SMD:R_0603_1608Metric_Pad0.98x0.95mm_HandSolder"
 			(at 176.022 121.92 90)
 			(effects
@@
 			(project "V101"
 				(path "/2bb6e42f-287e-4818-b6e1-26da2df0523c/365ddd10-1d92-4508-9f35-2b0988a801cb"
-					(reference "R703")
+					(reference "R702")
 					(unit 1)
 				)
@@
 			)
 		)
-		(property "Footprint" ""
+		(property "Footprint" "Resistor_SMD:R_0603_1608Metric_Pad0.98x0.95mm_HandSolder"
 			(at 176.022 50.8 90)
 			(effects
@@
 		(dnp no)
 		(fields_autoplaced yes)
-		(property "Reference" "#PWR0709"
+		(property "Reference" "#PWR0708"
 			(at 140.97 154.94 0)
 			(effects
@@
 			(project "V101"
 				(path "/2bb6e42f-287e-4818-b6e1-26da2df0523c/365ddd10-1d92-4508-9f35-2b0988a801cb"
-					(reference "#PWR0709")
+					(reference "#PWR0708")
 					(unit 1)
 				)
@@
 		(dnp no)
 		(fields_autoplaced yes)
-		(property "Reference" "C702"
+		(property "Reference" "C701"
 			(at 104.14 40.6399 0)
 			(effects
@@
 			)
 		)
-		(property "Footprint" ""
+		(property "Footprint" "Capacitor_SMD:C_0603_1608Metric_Pad1.08x0.95mm_HandSolder"
 			(at 101.2952 45.72 0)
 			(effects
@@
 			(project "V101"
 				(path "/2bb6e42f-287e-4818-b6e1-26da2df0523c/365ddd10-1d92-4508-9f35-2b0988a801cb"
-					(reference "C702")
+					(reference "C701")
 					(unit 1)
 				)
@@
 		(dnp no)
 		(fields_autoplaced yes)
-		(property "Reference" "#PWR0707"
+		(property "Reference" "#PWR0704"
 			(at 113.03 129.54 0)
 			(effects
@@
 			(project "V101"
 				(path "/2bb6e42f-287e-4818-b6e1-26da2df0523c/365ddd10-1d92-4508-9f35-2b0988a801cb"
-					(reference "#PWR0707")
+					(reference "#PWR0704")
 					(unit 1)
 				)
@@
 		(dnp no)
 		(fields_autoplaced yes)
-		(property "Reference" "C701"
+		(property "Reference" "C703"
 			(at 116.84 40.6399 0)
 			(effects
@@
 			)
 		)
-		(property "Footprint" ""
+		(property "Footprint" "Capacitor_SMD:C_0603_1608Metric_Pad1.08x0.95mm_HandSolder"
 			(at 113.9952 45.72 0)
 			(effects
@@
 			(project ""
 				(path "/2bb6e42f-287e-4818-b6e1-26da2df0523c/365ddd10-1d92-4508-9f35-2b0988a801cb"
-					(reference "C701")
+					(reference "C703")
 					(unit 1)
 				)
@@
 		(dnp no)
 		(fields_autoplaced yes)
-		(property "Reference" "#PWR0706"
+		(property "Reference" "#PWR0702"
 			(at 100.33 129.54 0)
 			(effects
@@
 			(project "V101"
 				(path "/2bb6e42f-287e-4818-b6e1-26da2df0523c/365ddd10-1d92-4508-9f35-2b0988a801cb"
-					(reference "#PWR0706")
+					(reference "#PWR0702")
 					(unit 1)
 				)
@@
 		(dnp no)
 		(fields_autoplaced yes)
-		(property "Reference" "#PWR0705"
+		(property "Reference" "#PWR0703"
 			(at 113.03 58.42 0)
 			(effects
@@
 			(project "V101"
 				(path "/2bb6e42f-287e-4818-b6e1-26da2df0523c/365ddd10-1d92-4508-9f35-2b0988a801cb"
-					(reference "#PWR0705")
+					(reference "#PWR0703")
 					(unit 1)
 				)
@@
 		(dnp no)
 		(fields_autoplaced yes)
-		(property "Reference" "C703"
+		(property "Reference" "C702"
 			(at 104.14 111.7599 0)
 			(effects
@@
 			)
 		)
-		(property "Footprint" ""
+		(property "Footprint" "Capacitor_SMD:C_0603_1608Metric_Pad1.08x0.95mm_HandSolder"
 			(at 101.2952 116.84 0)
 			(effects
@@
 			(project "V101"
 				(path "/2bb6e42f-287e-4818-b6e1-26da2df0523c/365ddd10-1d92-4508-9f35-2b0988a801cb"
-					(reference "C703")
+					(reference "C702")
 					(unit 1)
 				)
@@
 			)
 		)
-		(property "Footprint" ""
+		(property "Footprint" "Resistor_SMD:R_0603_1608Metric_Pad0.98x0.95mm_HandSolder"
 			(at 188.722 121.92 90)
 			(effects
@@
 			)
 		)
-		(property "Footprint" ""
+		(property "Footprint" "Capacitor_SMD:C_0603_1608Metric_Pad1.08x0.95mm_HandSolder"
 			(at 113.9952 116.84 0)
 			(effects
@@
 		(dnp no)
 		(fields_autoplaced yes)
-		(property "Reference" "#PWR0708"
+		(property "Reference" "#PWR0706"
 			(at 135.89 154.94 0)
 			(effects
@@
 			(project "V101"
 				(path "/2bb6e42f-287e-4818-b6e1-26da2df0523c/365ddd10-1d92-4508-9f35-2b0988a801cb"
-					(reference "#PWR0708")
+					(reference "#PWR0706")
 					(unit 1)
 				)
@@
 		(dnp no)
 		(fields_autoplaced yes)
-		(property "Reference" "R702"
+		(property "Reference" "R703"
 			(at 193.04 49.5299 0)
 			(effects
@@
 			)
 		)
-		(property "Footprint" ""
+		(property "Footprint" "Resistor_SMD:R_0603_1608Metric_Pad0.98x0.95mm_HandSolder"
 			(at 188.722 50.8 90)
 			(effects
@@
 			(project "V101"
 				(path "/2bb6e42f-287e-4818-b6e1-26da2df0523c/365ddd10-1d92-4508-9f35-2b0988a801cb"
-					(reference "R702")
+					(reference "R703")
 					(unit 1)
 				)
@@
 		(dnp no)
 		(fields_autoplaced yes)
-		(property "Reference" "#PWR0701"
+		(property "Reference" "#PWR0705"
 			(at 135.89 83.82 0)
 			(effects
@@
 			(project ""
 				(path "/2bb6e42f-287e-4818-b6e1-26da2df0523c/365ddd10-1d92-4508-9f35-2b0988a801cb"
-					(reference "#PWR0701")
+					(reference "#PWR0705")
 					(unit 1)
 				)
@@
 		(dnp no)
 		(fields_autoplaced yes)
-		(property "Reference" "#PWR0703"
+		(property "Reference" "#PWR0709"
 			(at 151.13 34.29 0)
 			(effects
@@
 			(project ""
 				(path "/2bb6e42f-287e-4818-b6e1-26da2df0523c/365ddd10-1d92-4508-9f35-2b0988a801cb"
-					(reference "#PWR0703")
+					(reference "#PWR0709")
 					(unit 1)
 				)
@@
 		(dnp no)
 		(fields_autoplaced yes)
-		(property "Reference" "#PWR0704"
+		(property "Reference" "#PWR0701"
 			(at 100.33 58.42 0)
 			(effects
@@
 			(project "V101"
 				(path "/2bb6e42f-287e-4818-b6e1-26da2df0523c/365ddd10-1d92-4508-9f35-2b0988a801cb"
-					(reference "#PWR0704")
+					(reference "#PWR0701")
 					(unit 1)
 				)
@@
 		(dnp no)
 		(fields_autoplaced yes)
-		(property "Reference" "#PWR0702"
+		(property "Reference" "#PWR0707"
 			(at 140.97 83.82 0)
 			(effects
@@
 			(project "V101"
 				(path "/2bb6e42f-287e-4818-b6e1-26da2df0523c/365ddd10-1d92-4508-9f35-2b0988a801cb"
-					(reference "#PWR0702")
-					(unit 1)
-				)
+					(reference "#PWR0707")
+					(unit 1)
+				)
