File: PCB/V101/Interface-RS485.kicad_sch (KiCad schematic)
At the start: 0 parts

Commit message: Updated PCB
Parts:
- added D801, D802: SMAJ7.0CA, Diode_SMD:D_SMA, symbol Diode:SMAJ7.0CA
- added J801: Conn_01x04, symbol Connector_Generic:Conn_01x04
- added R801, R802, R803, R804, R805, R806: 10R, symbol Device:R
- added U801: THVD1450D, Package_SO:SOIC-8_3.9x4.9mm_P1.27mm, symbol Interface_UART:THVD1450D
Connections:
- new net: R801.1, U801.6 (A)
- new net: D801.2 (A2), J801.2 (Pin_2), R801.2
- new net: R803.2, U801.1 (RO)
- new net: R804.2, U801.2 (~{RE})
- new net: R805.2, U801.3 (DE)
- new net: R806.2, U801.4 (DI)
- new net: R802.1, U801.7 (B)
- new net: D802.2 (A2), J801.3 (Pin_3), R802.2
- new net +5V: U801.8 (VCC)
- new net GND: D801.1 (A1), D802.1 (A1), J801.4 (Pin_4)
- new net USART1_DE_PIN: R805.1
- new net USART1_RE_PIN: R804.1
- new net USART1_RX_PIN: R803.1
- new net USART1_TX_PIN: R806.1
- new net VDD: J801.1 (Pin_1)

Commit message: Updated Layout
Parts:
- J801: footprint (none) -> Connector_JST:JST_PH_S4B-PH-K_1x04_P2.00mm_Horizontal
- R801: renamed from R803; footprint (none) -> Resistor_SMD:R_0603_1608Metric_Pad0.98x0.95mm_HandSolder
- R802: renamed from R804; footprint (none) -> Resistor_SMD:R_0603_1608Metric_Pad0.98x0.95mm_HandSolder
- R803: renamed from R805; footprint (none) -> Resistor_SMD:R_0603_1608Metric_Pad0.98x0.95mm_HandSolder
- R804: renamed from R806; footprint (none) -> Resistor_SMD:R_0603_1608Metric_Pad0.98x0.95mm_HandSolder
- R805: renamed from R801; footprint (none) -> Resistor_SMD:R_0603_1608Metric_Pad0.98x0.95mm_HandSolder
- R806: renamed from R802; footprint (none) -> Resistor_SMD:R_0603_1608Metric_Pad0.98x0.95mm_HandSolder
Changed lines of the file:
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@@
 		(on_board yes)
 		(dnp no)
-		(property "Reference" "R801"
+		(property "Reference" "R805"
 			(at 138.43 78.74 90)
 			(effects
@@
 			)
 		)
-		(property "Footprint" ""
+		(property "Footprint" "Resistor_SMD:R_0603_1608Metric_Pad0.98x0.95mm_HandSolder"
 			(at 138.43 80.518 90)
 			(effects
@@
 			(project ""
 				(path "/2bb6e42f-287e-4818-b6e1-26da2df0523c/39221d1a-c991-44a5-9f0e-70e43461fc41"
-					(reference "R801")
+					(reference "R805")
 					(unit 1)
 				)
@@
 			)
 		)
-		(property "Footprint" ""
+		(property "Footprint" "Connector_JST:JST_PH_S4B-PH-K_1x04_P2.00mm_Horizontal"
 			(at 193.04 80.01 0)
 			(effects
@@
 		(on_board yes)
 		(dnp no)
-		(property "Reference" "R803"
+		(property "Reference" "R801"
 			(at 97.79 81.28 90)
 			(effects
@@
 			)
 		)
-		(property "Footprint" ""
+		(property "Footprint" "Resistor_SMD:R_0603_1608Metric_Pad0.98x0.95mm_HandSolder"
 			(at 97.79 83.058 90)
 			(effects
@@
 			(project "V101"
 				(path "/2bb6e42f-287e-4818-b6e1-26da2df0523c/39221d1a-c991-44a5-9f0e-70e43461fc41"
-					(reference "R803")
+					(reference "R801")
 					(unit 1)
 				)
@@
 		(dnp no)
 		(fields_autoplaced yes)
-		(property "Reference" "#PWR0802"
+		(property "Reference" "#PWR0803"
 			(at 166.37 105.41 0)
 			(effects
@@
 			(project "V101"
 				(path "/2bb6e42f-287e-4818-b6e1-26da2df0523c/39221d1a-c991-44a5-9f0e-70e43461fc41"
-					(reference "#PWR0802")
+					(reference "#PWR0803")
 					(unit 1)
 				)
@@
 		(on_board yes)
 		(dnp no)
-		(property "Reference" "R802"
+		(property "Reference" "R806"
 			(at 138.43 83.82 90)
 			(effects
@@
 			)
 		)
-		(property "Footprint" ""
+		(property "Footprint" "Resistor_SMD:R_0603_1608Metric_Pad0.98x0.95mm_HandSolder"
 			(at 138.43 85.598 90)
 			(effects
@@
 			(project "V101"
 				(path "/2bb6e42f-287e-4818-b6e1-26da2df0523c/39221d1a-c991-44a5-9f0e-70e43461fc41"
-					(reference "R802")
+					(reference "R806")
 					(unit 1)
 				)
@@
 		(on_board yes)
 		(dnp no)
-		(property "Reference" "R806"
+		(property "Reference" "R804"
 			(at 97.79 91.44 90)
 			(effects
@@
 			)
 		)
-		(property "Footprint" ""
+		(property "Footprint" "Resistor_SMD:R_0603_1608Metric_Pad0.98x0.95mm_HandSolder"
 			(at 97.79 93.218 90)
 			(effects
@@
 			(project "V101"
 				(path "/2bb6e42f-287e-4818-b6e1-26da2df0523c/39221d1a-c991-44a5-9f0e-70e43461fc41"
-					(reference "R806")
+					(reference "R804")
 					(unit 1)
 				)
@@
 		(dnp no)
 		(fields_autoplaced yes)
-		(property "Reference" "#PWR0804"
+		(property "Reference" "#PWR0801"
 			(at 120.65 68.58 0)
 			(effects
@@
 			(project ""
 				(path "/2bb6e42f-287e-4818-b6e1-26da2df0523c/39221d1a-c991-44a5-9f0e-70e43461fc41"
-					(reference "#PWR0804")
+					(reference "#PWR0801")
 					(unit 1)
 				)
@@
 		(dnp no)
 		(fields_autoplaced yes)
-		(property "Reference" "#PWR0805"
+		(property "Reference" "#PWR0804"
 			(at 179.07 73.66 0)
 			(effects
@@
 			(project ""
 				(path "/2bb6e42f-287e-4818-b6e1-26da2df0523c/39221d1a-c991-44a5-9f0e-70e43461fc41"
-					(reference "#PWR0805")
+					(reference "#PWR0804")
 					(unit 1)
 				)
@@
 		(on_board yes)
 		(dnp no)
-		(property "Reference" "R805"
+		(property "Reference" "R803"
 			(at 97.79 86.36 90)
 			(effects
@@
 			)
 		)
-		(property "Footprint" ""
+		(property "Footprint" "Resistor_SMD:R_0603_1608Metric_Pad0.98x0.95mm_HandSolder"
 			(at 97.79 88.138 90)
 			(effects
@@
 			(project "V101"
 				(path "/2bb6e42f-287e-4818-b6e1-26da2df0523c/39221d1a-c991-44a5-9f0e-70e43461fc41"
-					(reference "R805")
+					(reference "R803")
 					(unit 1)
 				)
@@
 		(dnp no)
 		(fields_autoplaced yes)
-		(property "Reference" "#PWR0801"
+		(property "Reference" "#PWR0802"
 			(at 151.13 105.41 0)
 			(effects
@@
 			(project ""
 				(path "/2bb6e42f-287e-4818-b6e1-26da2df0523c/39221d1a-c991-44a5-9f0e-70e43461fc41"
-					(reference "#PWR0801")
+					(reference "#PWR0802")
 					(unit 1)
 				)
@@
 		(on_board yes)
 		(dnp no)
-		(property "Reference" "R804"
+		(property "Reference" "R802"
 			(at 97.79 83.82 90)
 			(effects
@@
 			)
 		)
-		(property "Footprint" ""
+		(property "Footprint" "Resistor_SMD:R_0603_1608Metric_Pad0.98x0.95mm_HandSolder"
 			(at 97.79 85.598 90)
 			(effects
@@
 			(project "V101"
 				(path "/2bb6e42f-287e-4818-b6e1-26da2df0523c/39221d1a-c991-44a5-9f0e-70e43461fc41"
-					(reference "R804")
+					(reference "R802")
 					(unit 1)
 				)
@@
 		(dnp no)
 		(fields_autoplaced yes)
-		(property "Reference" "#PWR0803"
+		(property "Reference" "#PWR0805"
 			(at 185.42 96.52 0)
 			(effects
@@
 			(project "V101"
 				(path "/2bb6e42f-287e-4818-b6e1-26da2df0523c/39221d1a-c991-44a5-9f0e-70e43461fc41"
-					(reference "#PWR0803")
-					(unit 1)
-				)
+					(reference "#PWR0805")
+					(unit 1)
+				)

Commit message: Updated PCB
Parts:
- added C801: 0.1uF, Capacitor_SMD:C_0603_1608Metric_Pad1.08x0.95mm_HandSolder, symbol Device:C
Connections:
- net +5V: now also C801.1
- net GND: now also U801.5 (GND), C801.2
