File: PCB/V101/V101.kicad_pcb (KiCad board)
At the start: 2 copper layers, 100 x 100 mm, 15 parts, among them U501 STM32G431CBUx

Commit message: Updated Layout
Parts:
- added C515: 100nF, Capacitor_SMD:C_0402_1005Metric_Pad0.74x0.62mm_HandSolder, F.Cu at (55.4, 72.9)
- added C516: 100nF, Capacitor_SMD:C_0402_1005Metric_Pad0.74x0.62mm_HandSolder, F.Cu at (55.4, 74.9)
- added C517: 100nF, Capacitor_SMD:C_0402_1005Metric_Pad0.74x0.62mm_HandSolder, F.Cu at (55.4, 76.9)
- added C601: 10uF, Capacitor_SMD:C_0603_1608Metric_Pad1.08x0.95mm_HandSolder, F.Cu at (126.2, 96.2)
- added C602: 0.1uF, Capacitor_SMD:C_0603_1608Metric_Pad1.08x0.95mm_HandSolder, F.Cu at (126.2, 94.4)
- added C603: 0.1uF, Capacitor_SMD:C_0603_1608Metric_Pad1.08x0.95mm_HandSolder, F.Cu at (121.0, 91.2)
- added C604: 22uF, Capacitor_SMD:C_0603_1608Metric_Pad1.08x0.95mm_HandSolder, F.Cu at (122.2, 100.0)
- added C605: 22uF, Capacitor_SMD:C_0603_1608Metric_Pad1.08x0.95mm_HandSolder, F.Cu at (122.2, 101.6)
- added C606: 22uF, Capacitor_SMD:C_0603_1608Metric_Pad1.08x0.95mm_HandSolder, F.Cu at (124.6, 87.0)
- added C701: 100nF, Capacitor_SMD:C_0603_1608Metric_Pad1.08x0.95mm_HandSolder, F.Cu at (129.0, 81.7)
- added C702: 100nF, Capacitor_SMD:C_0603_1608Metric_Pad1.08x0.95mm_HandSolder, F.Cu at (168.3, 29.3)
- added C703: 100nF, Capacitor_SMD:C_0603_1608Metric_Pad1.08x0.95mm_HandSolder, F.Cu at (127.6, 77.7)
- added C704: 100nF, Capacitor_SMD:C_0603_1608Metric_Pad1.08x0.95mm_HandSolder, F.Cu at (168.3, 34.3)
- added C901: 4700pF, Capacitor_SMD:C_0603_1608Metric_Pad1.08x0.95mm_HandSolder, F.Cu at (150.2, 114.6)
- added C902: 0.1uF, Capacitor_SMD:C_0603_1608Metric_Pad1.08x0.95mm_HandSolder, F.Cu at (150.2, 103.6)
- added D801: SMAJ7.0CA, Diode_SMD:D_SMA, F.Cu at (124.8, 114.6)
- added D802: SMAJ7.0CA, Diode_SMD:D_SMA, F.Cu at (135.0, 114.6)
- added D901: SMAJ7.0CA, Diode_SMD:D_SMA, F.Cu at (155.0, 114.6)
- added D902: SMAJ7.0CA, Diode_SMD:D_SMA, F.Cu at (145.4, 114.6)
- added G***: LOGO, Blackshield_Engineering:Company Logo, B.Cu at (139.8, 91.6)
- added H1001: MountingHole, MountingHole:MountingHole_3.2mm_M3, F.Cu at (119.0, 79.0)
- added H1002: MountingHole, MountingHole:MountingHole_3.2mm_M3, F.Cu at (119.0, 121.0)
- added H1003: MountingHole, MountingHole:MountingHole_3.2mm_M3, F.Cu at (161.0, 121.0)
- added H1004: MountingHole, MountingHole:MountingHole_3.2mm_M3, F.Cu at (161.0, 79.0)
- added J801: Conn_01x04, Connector_JST:JST_PH_S4B-PH-K_1x04_P2.00mm_Horizontal, F.Cu at (127.0, 118.5)
- added J901: Conn_01x04, Connector_JST:JST_PH_S4B-PH-K_1x04_P2.00mm_Horizontal, F.Cu at (147.2, 118.4)
- added L601: 10uH, Inductor_SMD:L_APV_ANR5045, F.Cu at (121.2, 96.2)
- added R501: 4.7K, Resistor_SMD:R_0603_1608Metric_Pad0.98x0.95mm_HandSolder, F.Cu at (100.1, 68.0)
- added R502: 4.7K, Resistor_SMD:R_0603_1608Metric_Pad0.98x0.95mm_HandSolder, F.Cu at (100.1, 70.5)
- added R503: 4.7K, Resistor_SMD:R_0603_1608Metric_Pad0.98x0.95mm_HandSolder, F.Cu at (100.1, 73.0)
- added R601: 511K, Resistor_SMD:R_0603_1608Metric_Pad0.98x0.95mm_HandSolder, F.Cu at (127.2, 91.3)
- added R602: 105K, Resistor_SMD:R_0603_1608Metric_Pad0.98x0.95mm_HandSolder, F.Cu at (127.2, 87.9)
- added R603: R, Resistor_SMD:R_0603_1608Metric_Pad0.98x0.95mm_HandSolder, F.Cu at (117.2, 97.4)
- added R604: R, Resistor_SMD:R_0603_1608Metric_Pad0.98x0.95mm_HandSolder, F.Cu at (117.2, 93.6)
- added R605: R, Resistor_SMD:R_0603_1608Metric_Pad0.98x0.95mm_HandSolder, F.Cu at (117.2, 89.8)
- added R701: 4.7k, Resistor_SMD:R_0603_1608Metric_Pad0.98x0.95mm_HandSolder, F.Cu at (132.6, 81.7)
- added R702: 4.7k, Resistor_SMD:R_0603_1608Metric_Pad0.98x0.95mm_HandSolder, F.Cu at (193.5, 5.16)
- added R703: 4.7k, Resistor_SMD:R_0603_1608Metric_Pad0.98x0.95mm_HandSolder, F.Cu at (133.6, 78.1)
- added R704: 4.7k, Resistor_SMD:R_0603_1608Metric_Pad0.98x0.95mm_HandSolder, F.Cu at (193.5, 10.2)
- added R801: 10R, Resistor_SMD:R_0603_1608Metric_Pad0.98x0.95mm_HandSolder, F.Cu at (257.2, 53.9)
- added R802: 10R, Resistor_SMD:R_0603_1608Metric_Pad0.98x0.95mm_HandSolder, F.Cu at (257.2, 56.4)
- added R803: 10R, Resistor_SMD:R_0603_1608Metric_Pad0.98x0.95mm_HandSolder, F.Cu at (257.2, 58.9)
- added R804: 10R, Resistor_SMD:R_0603_1608Metric_Pad0.98x0.95mm_HandSolder, F.Cu at (257.2, 61.4)
- added R805: 10R, Resistor_SMD:R_0603_1608Metric_Pad0.98x0.95mm_HandSolder, F.Cu at (127.6, 111.0)
- added R806: 10R, Resistor_SMD:R_0603_1608Metric_Pad0.98x0.95mm_HandSolder, F.Cu at (132.2, 111.0)
- added R901: 60R, Resistor_SMD:R_0603_1608Metric_Pad0.98x0.95mm_HandSolder, F.Cu at (153.0, 111.0)
- added R902: 60R, Resistor_SMD:R_0603_1608Metric_Pad0.98x0.95mm_HandSolder, F.Cu at (147.4, 111.2)
- added U601: TPS54302, Package_TO_SOT_SMD:SOT-23-6, F.Cu at (123.8, 91.0)
- added U701: BME280, Package_LGA:Bosch_LGA-8_2.5x2.5mm_P0.65mm_ClockwisePinNumbering, F.Cu at (130.6, 79.2)
- added U702: BME280, Package_LGA:Bosch_LGA-8_2.5x2.5mm_P0.65mm_ClockwisePinNumbering, F.Cu at (196.2, 38.1)
- added U801: THVD1450D, Package_SO:SOIC-8_3.9x4.9mm_P1.27mm, F.Cu at (129.8, 105.2)
- added U901: MCP2557FD-xMF, Package_DFN_QFN:DFN-8-1EP_3x3mm_P0.65mm_EP1.55x2.4mm, F.Cu at (150.2, 107.2)
- C509: value 4.7uF -> 100nF
- C512: value 100nF -> 4.7uF
- U501: value STM32G431CBUx -> STM32G431CBTx; footprint Package_DFN_QFN:QFN-48-1EP_7x7mm_P0.5mm_EP5.6x5.6mm -> Package_QFP:LQFP-48_7x7mm_P0.5mm
- moved C513 101.6 mm to (158.1, 87.0), turned to 90 degrees
- moved C512 99.6 mm to (157.0, 87.0), turned to 90 degrees
- moved C501 97.2 mm to (48.9, 72.9), turned to 0 degrees
- moved C509 96.1 mm to (52.2, 78.8), turned to 0 degrees
- moved C502 95.6 mm to (48.9, 74.9), turned to 0 degrees
- moved C508 95.6 mm to (52.2, 76.9)
- moved C511 95.2 mm to (157.1, 97.0)
- moved C510 94.6 mm to (52.2, 80.8), turned to 0 degrees
- moved U501 15.1 mm to (152.6, 91.6)
- moved C506 14.8 mm to (148.1, 87.2)
- moved C505 14.8 mm to (148.1, 86.2)
- moved C504 14.5 mm to (154.1, 99.4)
- moved C503 14.4 mm to (155.1, 99.4)
- moved C507 11.6 mm to (157.1, 96.0)
Connections:
- C508 pad 1: +3V3 -> /MCU/BUTTON1
- C509 pad 1: +3V3 -> /MCU/BUTTON2
- C510 pad 1: +3V3 -> /MCU/BUTTON3
- C511 pad 1: /MCU/HSE_IN -> +3V3
- C512 pad 1: /MCU/HSE_OUT -> +3V3
- C513 pad 1: /MCU/LSE_IN -> +3V3
- C514 pad 1: /MCU/LSE_OUT -> /MCU/LSE_IN
- U501 pad 1: unconnected-(U501-VBAT-Pad1) -> +3V3
- U501 pad 19: unconnected-(U501-PB2-Pad19) -> GND
- U501 pad 2: /MCU/LSE_IN -> unconnected-(U501-PC13-Pad2)
- U501 pad 23: +3V3 -> GND
- U501 pad 24: unconnected-(U501-PB11-Pad24) -> +3V3
- U501 pad 3: /MCU/LSE_OUT -> /MCU/LSE_IN
- U501 pad 35: +3V3 -> GND
- U501 pad 36: unconnected-(U501-PA13-Pad36) -> +3V3
- U501 pad 4: unconnected-(U501-PC15-Pad4) -> /MCU/LSE_OUT
- U501 pad 47: unconnected-(U501-PB9-Pad47) -> GND
Routing:
- net Net-(D901-A2): track 0.00 -> 11.5 mm
- net Net-(D902-A2): track 0.00 -> 11.4 mm
- net +3V3: track 0.00 -> 11.2 mm
- net Net-(D801-A2): track 0.00 -> 7.88 mm
- net Net-(D802-A2): track 0.00 -> 7.80 mm
- net /MCU/LSE_OUT: track 6.71 -> 0.00 mm
- net /MCU/LSE_IN: track 6.67 -> 0.00 mm
- net /MCU/HSE_OUT: track 6.67 -> 0.00 mm
- net /MCU/HSE_IN: track 6.62 -> 0.00 mm
- net +5V: track 0.00 -> 6.56 mm
- net Net-(U601-SW): track 0.00 -> 6.27 mm
- net Net-(U601-EN): track 0.00 -> 6.13 mm
- net GND: track 0.00 -> 5.99 mm, vias 0 -> 3
- net V_IN: track 0.00 -> 4.99 mm
- net Net-(U801-B): track 0.00 -> 3.14 mm
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Other:
- board size 100 x 100 mm -> 50 x 50 mm

Commit message: Updated PCB
Parts:
- added C801: 0.1uF, Capacitor_SMD:C_0603_1608Metric_Pad1.08x0.95mm_HandSolder, F.Cu at (134.7, 108.2)
- moved R804 135.7 mm to (127.0, 99.6), turned to -90 degrees
- moved R803 134.7 mm to (128.8, 99.6), turned to -90 degrees
- moved R802 133.8 mm to (130.6, 99.6), turned to -90 degrees
- moved R801 132.9 mm to (132.4, 99.6), turned to -90 degrees
- moved R702 87.4 mm to (152.0, 82.1)
- moved C501 86.8 mm to (-36.8, 86.1)
- moved C502 86.8 mm to (-36.8, 88.1)
- moved C508 86.8 mm to (-33.6, 90.1)
- moved C509 86.8 mm to (-33.6, 92.0)
- moved C510 86.8 mm to (-33.6, 94.0)
- moved C514 86.8 mm to (-19.5, 146.2)
- moved C515 86.8 mm to (-30.4, 86.1)
- moved C516 86.8 mm to (-30.4, 88.1)
- moved C517 86.8 mm to (-30.4, 90.1)
- moved R502 86.8 mm to (14.3, 83.7)
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Connections:
- U801 pad 5: unconnected-(U801-GND-Pad5) -> GND
Routing:
- net +5V: track 6.56 -> 17.8 mm
- net GND: track 5.99 -> 9.71 mm
- net I2C1_SCL: track 3.03 -> 6.19 mm
- net I2C1_SDA: track 2.19 -> 4.51 mm
